File: Rotary-Dial-Tester-Adapter.kicad_sch (KiCad schematic)
At the start: 14 parts, among them J1 DE9_Receptacle, J2 7770, J3 7770, J4 7770, J5 7770, J6 Conn_01x04_Pin

Commit message: Adds project license and metadata
Adds a "Permission Required License" and copyright notice.

Updates the schematic and PCB files to include a title block with project metadata and license information.
This ensures proper attribution and clarifies usage restrictions.
Other:
- title: (none) -> Rotary Dial Tester Adapter
Changed lines of the file:
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@@
 (kicad_sch
-	(version 20231120)
+	(version 20250114)
 	(generator "eeschema")
-	(generator_version "8.0")
+	(generator_version "9.0")
 	(paper "A4")
+	(title_block
+		(title "Rotary Dial Tester Adapter")
+		(date "2026-01-12")
+		(rev "1.3")
+		(comment 1 "Permission Required License")
+		(comment 2 "Copyright (c) 2026 Andre Fiedler. All rights reserved.")
+		(comment 3 "Use requires written permission; see LICENSE.")
+		(comment 4 "Attribution: project name \"Rotary Dial Tester\" + notice.")
+	)
 	(junction
 		(at 43.18 50.8)
@@
 	(label "BRAUN"
 		(at 63.5 77.47 0)
-		(fields_autoplaced yes)
 		(effects
 			(font
@@
 	(label "WEIß"
 		(at 76.2 77.47 0)
-		(fields_autoplaced yes)
 		(effects
 			(font
@@
 	(label "GRÜN"
 		(at 50.8 77.47 0)
-		(fields_autoplaced yes)
 		(effects
 			(font
@@
 	(label "GELB"
 		(at 38.1 77.47 0)
-		(fields_autoplaced yes)
 		(effects
 			(font
@@
 		)
 	)
+	(embedded_fonts no)
 )
